Commit message: changes

File: Section12_Build_the_Robot/bumperbot_ws/src/bumperbot_description/urdf/bumperbot.urdf.xacro (robot description, xacro)
@@ -175,3 +175,18 @@
     <axis xyz="0 0 0" />
   </joint>
+<ros2_control name="BumperbotSystem" type="system">
+  <hardware>
+    <plugin>bumperbot_firmware/BumperbotSystemHardware</plugin>
+  </hardware>
+  <joint name="wheel_left_joint">
+    <command_interface name="velocity"/>
+    <state_interface name="velocity"/>
+    <state_interface name="position"/>
+  </joint>
+  <joint name="wheel_right_joint">
+    <command_interface name="velocity"/>
+    <state_interface name="velocity"/>
+    <state_interface name="position"/>
+  </joint>
+</ros2_control>
 </robot>

File: Section12_Build_the_Robot/bumperbot_ws/src/bumperbot_description/urdf/bumperbot_ros2_control.xacro (robot description, xacro)
@@ -21,5 +21,5 @@
             <hardware>
                 <plugin>bumperbot_firmware/BumperbotInterface</plugin>
-                <param name="port">/dev/ttyUSB0</param>
+                <param name="port">/dev/ttyACM0</param>
             </hardware>
         </xacro:unless>

Commit message: working, just to fast

File: Section12_Build_the_Robot/bumperbot_ws/src/bumperbot_description/urdf/bumperbot.urdf.xacro (robot description, xacro)
@@ -175,18 +175,3 @@
     <axis xyz="0 0 0" />
   </joint>
-<ros2_control name="BumperbotSystem" type="system">
-  <hardware>
-    <plugin>bumperbot_firmware/BumperbotSystemHardware</plugin>
-  </hardware>
-  <joint name="wheel_left_joint">
-    <command_interface name="velocity"/>
-    <state_interface name="velocity"/>
-    <state_interface name="position"/>
-  </joint>
-  <joint name="wheel_right_joint">
-    <command_interface name="velocity"/>
-    <state_interface name="velocity"/>
-    <state_interface name="position"/>
-  </joint>
-</ros2_control>
 </robot>

File: Section12_Build_the_Robot/bumperbot_ws/src/bumperbot_description/urdf/bumperbot_ros2_control.xacro (robot description, xacro)
@@ -1,44 +1,45 @@
 <?xml version="1.0"?>
 <robot xmlns:xacro="http://www.ros.org/wiki/xacro" name="bumperbot">
-    <ros2_control name="RobotSystem" type="system">
-        <!-- ros2_control Gazebo -->
-        <xacro:if value="$(arg is_sim)">
-            <!-- ROS 2 Humble -->
-            <xacro:if value="$(arg is_ignition)">
-                <hardware>
-                    <plugin>ign_ros2_control/IgnitionSystem</plugin>
-                </hardware>
-            </xacro:if>
-            <!-- ROS 2 Iron or above -->
-            <xacro:unless value="$(arg is_ignition)">
-                <hardware>
-                    <plugin>gz_ros2_control/GazeboSimSystem</plugin>
-                </hardware>
-            </xacro:unless>
-        </xacro:if>
-        <!-- ros2_control Real Robot -->
-        <xacro:unless value="$(arg is_sim)">
-            <hardware>
-                <plugin>bumperbot_firmware/BumperbotInterface</plugin>
-                <param name="port">/dev/ttyACM0</param>
-            </hardware>
-        </xacro:unless>
-        <!-- ros2_control Common Interfaces -->
-        <joint name="wheel_right_joint">
-            <command_interface name="velocity">
-              <param name="min">-1</param>
-              <param name="max">1</param>
-            </command_interface>
-            <state_interface name="position" />
-            <state_interface name="velocity" />
-        </joint>
-        <joint name="wheel_left_joint">
-            <command_interface name="velocity">
-              <param name="min">-1</param>
-              <param name="max">1</param>
-            </command_interface>
-            <state_interface name="position" />
-            <state_interface name="velocity" />
-        </joint>
-    </ros2_control>
+  <!-- ros2_control Interface -->
+  <ros2_control name="RobotSystem" type="system">
+    <!-- Simulation hardware -->
+    <xacro:if value="$(arg is_sim)">
+      <!-- Humble with Ignition -->
+      <xacro:if value="$(arg is_ignition)">
+        <hardware>
+          <plugin>ign_ros2_control/IgnitionSystem</plugin>
+        </hardware>
+      </xacro:if>
+      <!-- Humble with Gazebo Classic -->
+      <xacro:unless value="$(arg is_ignition)">
+        <hardware>
+          <plugin>gz_ros2_control/GazeboSimSystem</plugin>
+        </hardware>
+      </xacro:unless>
+    </xacro:if>
+    <!-- Real robot hardware -->
+    <xacro:unless value="$(arg is_sim)">
+      <hardware>
+        <plugin>bumperbot_firmware/BumperbotInterface</plugin>
+        <param name="port">/dev/ttyACM0</param>
+      </hardware>
+    </xacro:unless>
+    <!-- Wheel joint interfaces -->
+    <joint name="wheel_right_joint">
+      <command_interface name="velocity">
+        <param name="min">-1.0</param>
+        <param name="max">1.0</param>
+      </command_interface>
+      <state_interface name="position" />
+      <state_interface name="velocity" />
+    </joint>
+    <joint name="wheel_left_joint">
+      <command_interface name="velocity">
+        <param name="min">-1.0</param>
+        <param name="max">1.0</param>
+      </command_interface>
+      <state_interface name="position" />
+      <state_interface name="velocity" />
+    </joint>
+  </ros2_control>
 </robot>
